Commit message: -Fix material name

File: urdf/artag.urdf.xacro (robot description, xacro)
@@ -58,5 +58,5 @@
     </gazebo>
     <gazebo reference="${name}_background_link">
-      <material>White</material>
+      <material>Gazebo/White</material>
       <!--
       <turnGravityOff>false</turnGravityOff>
